File: hardware/Comms/Radio Board.brd (EAGLE design)
At the start: 90.2 x 95.5 mm, 1 part

Commit message: Completed radio boards
Parts:
- added J1: MOLEX_503763-0491MOLEX_503763-0491_0_0, Molex - 503763-0491:MOLEX_503763-0491_0
- added J2: MOLEX_503763-0291MOLEX_503763-0291_0_0, Molex - 503763-0291:MOLEX_503763-0291_0
- added J3: MCX-J-P-H-RA-TH1, MCX-J-P-H-RA-TH1:SAMTEC_MCX-J-P-H-RA-TH1
- added R1, R2: 1M, HSFL_Main_Library:0805
- added U1: LI-3_RADIO, Lithium-3 Radio:LI-3_RADIO
- added U2: RFM98W-433S2, RFM98:RFM98W-433S2
Connections:
- new net 3V3_RADIO_OUT: U1.5
- new net ANT: J3.1, U2.9
- new net CONFIG_1: U1.14
- new net CONFIG_2: U1.13
- new net DIO0: J2.2, U2.14
- new net DIO1: U2.15
- new net DIO2: U2.16
- new net DIO3: U2.11
- new net DIO4: U2.12
- new net DIO5: U2.7
- new net EXTERNAL: U1.12
- new net GND: H1.2.14, H1.2.17, H1.2.29, H1.2.30, H1.2.32, H1.2.47, H1.2.48, H1.2.7, H1.2.9, J1.2, J1.5, J1.6, J2.3, J2.4, J3.S1, J3.S2, J3.S3, J3.S4, R1.2, R2.1, U1.4, U2.1, U2.10, U2.8
- new net GPIO_A: U1.11
- new net GPIO_B: U1.10
- new net LI-3_RST: U1.3
- new net N$1: H1.P$4, R2.2
- new net RFM_RST: J2.1, U2.6
- new net RF_GND: R1.1, U1.15, U1.8, U1.9
- new net RX_UART: J1.3, U1.2
- new net SPI1_D0: H1.2.2, U2.3
- new net SPI1_D1: H1.2.3, U2.2
- new net SPI1_SCLK: H1.2.1, U2.4
- new net SW_3V3_2: H1.2.20, U2.13
- new net TX_UART: J1.4, U1.1
- new net T_CS1: H1.2.4, U2.5
- new net V_AMP: J1.1, U1.6, U1.7
Routing:
- net V_AMP: track 0.00 -> 61.2 mm
- net RFM_RST: track 0.00 -> 48.5 mm
- net SW_3V3_2: track 0.00 -> 40.1 mm
- net T_CS1: track 0.00 -> 40.1 mm
- net DIO0: track 0.00 -> 35.7 mm
- net RF_GND: track 0.00 -> 28.2 mm
- net SPI1_D0: track 0.00 -> 20.0 mm
- net SPI1_SCLK: track 0.00 -> 18.4 mm
- net SPI1_D1: track 0.00 -> 17.2 mm
- net RX_UART: track 0.00 -> 16.0 mm
- net TX_UART: track 0.00 -> 12.8 mm
- net ANT: track 0.00 -> 12.4 mm
- net N$1: track 0.00 -> 6.01 mm
- added copper zone on layer 1, net GND
- added copper zone on layer 16, net GND
